Commit message: expand urdf link joint limits

File: projects/urdf_two_joint_arm_demo/models/two_joint_arm.urdf (robot description, URDF)
Before this commit: robot two_joint_arm, 3 links, 2 joints
Links:
- added link tool0, mass 0.2; collision box size=0.08 0.08 0.08; visual box size=0.08 0.08 0.08
- link base_link: mass None -> 4.0; geometry collision box size=0.30 0.30 0.10; visual box size=0.30 0.30 0.10
- link elbow_link: mass None -> 1.0; geometry collision box size=0.40 0.05 0.05; visual box size=0.40 0.05 0.05
- link shoulder_link: mass None -> 1.6; geometry collision box size=0.50 0.06 0.06; visual box size=0.50 0.06 0.06
Joints:
- added joint tool_mount_joint: type fixed, parent elbow_link, child tool0, origin xyz=0.40 0 0 rpy=0 0 0

Commit message: add tf sensor frames and gazebo smoke

File: projects/urdf_two_joint_arm_demo/models/two_joint_arm.urdf (robot description, URDF)
Before this commit: robot two_joint_arm, 4 links, 3 joints
Links:
- added link imu_link, mass 0.05; collision box size=0.05 0.04 0.02; visual box size=0.05 0.04 0.02
Joints:
- added joint imu_mount_joint: type fixed, parent elbow_link, child imu_link, origin xyz=0.25 0 0.08 rpy=0 0 0
